File: Hardware/JammerESP.kicad_sch (KiCad schematic)
At the start: 21 parts, among them J1 NRF24L01, J2 NRF24L01, SW1 SW_Push, SW2 SW_Push, SW3 SW_Push, SW4 SW_Push, U1 ESP32-DEVKIT-V1, U2 DM-OLED096-636, U3 AMS1117-3.3, U4 AMS1117-3.3

Commit message: add pcb design
Parts:
- removed TP1: TX0, symbol Connector:TestPoint_Probe
- removed TP2: RX0, symbol Connector:TestPoint_Probe
- removed TP3: GND_CON, symbol Connector:TestPoint_Probe
- added J3: Conn_01x03_Socket, Connector_PinHeader_2.54mm:PinHeader_1x03_P2.54mm_Vertical, symbol Connector:Conn_01x03_Socket
- C1, C2, C3, C4, C5, C6, C7, C8: footprint (none) -> Capacitor_SMD:C_1206_3216Metric_Pad1.33x1.80mm_HandSolder
- J1, J2: footprint (none) -> Connector_PinHeader_2.54mm:PinHeader_2x04_P2.54mm_Vertical
- SW1: value SW_Push -> UP; footprint (none) -> Footprints:SW_BUTT-2
- SW2: value SW_Push -> DOWN; footprint (none) -> Footprints:SW_BUTT-2
- SW3: value SW_Push -> LEFT; footprint (none) -> Footprints:SW_BUTT-2
- SW4: value SW_Push -> RIGHT; footprint (none) -> Footprints:SW_BUTT-2
Connections:
- net GND: now also J3.3 (Pin_3)
- net at U1.12 (RX0): now also J3.1 (Pin_1)
- net at U1.13 (TX0): now also J3.2 (Pin_2)

Commit message: update routes
Connections:
- net DOWN: now also U1.23 (D25); no longer U1.21 (D32)
- net UP: now also U1.21 (D32); no longer U1.23 (D25)
Changed lines of the file:
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@@
 	)
 	(label "DOWN"
-		(at 128.27 62.23 0)
+		(at 128.27 54.61 0)
 		(effects
 			(font
@@
 	)
 	(label "UP"
-		(at 128.27 54.61 0)
+		(at 128.27 62.23 0)
 		(effects
 			(font
